Commit message: fixup! WIP XYZT robot

File: pnp_robot_description/urdf/pnp_robot.urdf (robot description, URDF)
Before this commit: robot pnp_robot, 8 links, 7 joints
Joints:
- removed joint theta_joint
- removed joint x_joint
- removed joint y_joint
- removed joint z_joint
- added joint theta: type revolute, parent y_link, child theta_link, origin xyz=0 0.1 0 rpy=0 0 0, axis 0 0 1, limit lower=-3.14159 upper=3.14159 effort=50 velocity=2.0
- added joint x: type prismatic, parent z_link, child x_link, origin xyz=0 0 0.1 rpy=0 0 0, axis 1 0 0, limit lower=-0.5 upper=0.5 effort=100 velocity=1.0
- added joint y: type prismatic, parent x_link, child y_link, origin xyz=0.1 0 0 rpy=0 0 0, axis 0 1 0, limit lower=-0.5 upper=0.5 effort=100 velocity=1.0
- added joint z: type prismatic, parent base_link, child z_link, origin xyz=0 0 0.05 rpy=0 0 0, axis 0 0 1, limit lower=0 upper=1.0 effort=100 velocity=1.0
